File: KiCad - 3S 1.0/LedBoard/LedBoard.kicad_sch (KiCad schematic)
At the start: 15 parts, among them J1 Conn_01x02, SW1 SW_SPST, U1 TPS565208

Commit message: Finished up LED PCB and made some small tweaks and fixes to main board.
Parts:
- D1, D2, D3: value GW CSSRM3.CM-MFN4-A232-1-L -> GW CSSRM1.BM
- R1: value 10K 0805 -> Value: 10K 0805
Connections:
- net GND: now also D1.3 (GND), D2.3 (GND), D3.3 (GND)
Changed lines of the file:
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@@
 (kicad_sch (version 20230121) (generator eeschema)
   (paper "A4")
+  (junction (at 103.505 67.31) (diameter 0) (color 0 0 0 0)
+  )
   (junction (at 114.3 41.275) (diameter 0) (color 0 0 0 0)
   )
   (junction (at 120.65 48.895) (diameter 0) (color 0 0 0 0)
   )
+  (junction (at 122.555 75.565) (diameter 0) (color 0 0 0 0)
+  )
   (junction (at 78.74 55.245) (diameter 0) (color 0 0 0 0)
   )
@@
   (junction (at 49.53 41.275) (diameter 0) (color 0 0 0 0)
   )
-  (junction (at 103.505 66.675) (diameter 0) (color 0 0 0 0)
-  )
   (junction (at 128.27 65.405) (diameter 0) (color 0 0 0 0)
   )
   (junction (at 120.65 41.275) (diameter 0) (color 0 0 0 0)
   )
+  (junction (at 103.505 60.96) (diameter 0) (color 0 0 0 0)
+  )
   (junction (at 128.27 59.055) (diameter 0) (color 0 0 0 0)
   )
@@
   (junction (at 99.06 41.275) (diameter 0) (color 0 0 0 0)
   )
-  (junction (at 103.505 60.325) (diameter 0) (color 0 0 0 0)
+  (junction (at 122.555 69.215) (diameter 0) (color 0 0 0 0)
   )
   (wire (pts (xy 128.27 41.275) (xy 128.27 59.055))
     (stroke (width 0) (type default))
   )
+  (wire (pts (xy 122.555 62.865) (xy 122.555 69.215))
+    (stroke (width 0) (type default))
+  )
+  (wire (pts (xy 122.555 69.215) (xy 122.555 75.565))
+    (stroke (width 0) (type default))
+  )
   (wire (pts (xy 49.53 48.895) (xy 49.53 47.625))
     (stroke (width 0) (type default))
@@
     (stroke (width 0) (type default))
   )
+  (wire (pts (xy 122.555 69.215) (xy 120.65 69.215))
+    (stroke (width 0) (type default))
+  )
   (wire (pts (xy 53.34 48.895) (xy 53.34 47.625))
     (stroke (width 0) (type default))
@@
     (stroke (width 0) (type default))
   )
-  (wire (pts (xy 103.505 66.675) (xy 103.505 73.025))
-    (stroke (width 0) (type default))
-  )
   (wire (pts (xy 120.65 41.275) (xy 114.3 41.275))
     (stroke (width 0) (type default))
@@
     (stroke (width 0) (type default))
   )
-  (wire (pts (xy 103.505 60.325) (xy 103.505 66.675))
-    (stroke (width 0) (type default))
-  )
   (wire (pts (xy 53.34 41.275) (xy 53.34 42.545))
     (stroke (width 0) (type default))
@@
     (stroke (width 0) (type default))
   )
-  (wire (pts (xy 105.41 60.325) (xy 103.505 60.325))
+  (wire (pts (xy 105.41 60.96) (xy 103.505 60.96))
+    (stroke (width 0) (type default))
+  )
+  (wire (pts (xy 103.505 60.96) (xy 103.505 67.31))
     (stroke (width 0) (type default))
   )
@@
     (stroke (width 0) (type default))
   )
+  (wire (pts (xy 122.555 75.565) (xy 120.65 75.565))
+    (stroke (width 0) (type default))
+  )
   (wire (pts (xy 114.3 41.275) (xy 106.68 41.275))
     (stroke (width 0) (type default))
@@
     (stroke (width 0) (type default))
   )
+  (wire (pts (xy 103.505 67.31) (xy 103.505 73.66))
+    (stroke (width 0) (type default))
+  )
   (wire (pts (xy 114.3 43.815) (xy 114.3 41.275))
     (stroke (width 0) (type default))
   )
-  (wire (pts (xy 103.505 46.355) (xy 103.505 60.325))
+  (wire (pts (xy 103.505 46.355) (xy 103.505 60.96))
     (stroke (width 0) (type default))
   )
@@
     (stroke (width 0) (type default))
   )
+  (wire (pts (xy 122.555 62.865) (xy 120.65 62.865))
+    (stroke (width 0) (type default))
+  )
   (wire (pts (xy 60.96 41.275) (xy 68.58 41.275))
     (stroke (width 0) (type default))
   )
-  (wire (pts (xy 105.41 73.025) (xy 103.505 73.025))
+  (wire (pts (xy 105.41 73.66) (xy 103.505 73.66))
     (stroke (width 0) (type default))
   )
@@
     (stroke (width 0) (type default))
   )
+  (wire (pts (xy 122.555 75.565) (xy 122.555 78.74))
+    (stroke (width 0) (type default))
+  )
   (wire (pts (xy 57.15 41.275) (xy 57.15 42.545))
     (stroke (width 0) (type default))
@@
     (stroke (width 0) (type default))
   )
-  (wire (pts (xy 105.41 66.675) (xy 103.505 66.675))
+  (wire (pts (xy 105.41 67.31) (xy 103.505 67.31))
     (stroke (width 0) (type default))
   )
@@
       (effects (font (size 1.27 1.27)))
     )
-    (property "Value" "GW CSSRM3.CM-MFN4-A232-1-L" (at 113.03 62.865 0)
+    (property "Value" "GW CSSRM1.BM" (at 113.03 62.865 0)
       (effects (font (size 1.27 1.27)) hide)
     )
@@
         (path "/d80cef19-75ee-4cfe-8d31-e56b6cad8d97"
           (reference "C105") (unit 1)
+        )
+      )
+    )
+  )
+  (symbol (lib_id "power:GND") (at 122.555 78.74 0) (unit 1)
+    (in_bom yes) (on_board yes) (dnp no) (fields_autoplaced)
+    (property "Reference" "#PWR05" (at 122.555 85.09 0)
+      (effects (font (size 1.27 1.27)) hide)
+    )
+    (property "Value" "GND" (at 122.555 83.185 0)
+      (effects (font (size 1.27 1.27)))
+    )
+    (property "Footprint" "" (at 122.555 78.74 0)
+      (effects (font (size 1.27 1.27)) hide)
+    )
+    (property "Datasheet" "" (at 122.555 78.74 0)
+      (effects (font (size 1.27 1.27)) hide)
+    )
+    (pin "1")
+    (instances
+      (project "LedBoard"
+        (path "/7007eb9b-f827-4e2f-a1f8-279aa4f63030"
+          (reference "#PWR05") (unit 1)
         )
       )
@@
   (symbol (lib_id "GW CSSRM3:GW_CSSRM3") (at 113.03 57.785 0) (mirror y) (unit 1)
     (in_bom yes) (on_board yes) (dnp no)
-    (property "Reference" "D1" (at 106.426 57.023 0)
-      (effects (font (size 1.27 1.27)))
-    )
-    (property "Value" "GW CSSRM3.CM-MFN4-A232-1-L" (at 113.03 56.515 0)
+    (property "Reference" "D1" (at 119.634 57.023 0)
+      (effects (font (size 1.27 1.27)))
+    )
+    (property "Value" "GW CSSRM1.BM" (at 113.03 56.515 0)
       (effects (font (size 1.27 1.27)) hide)
     )
@@
       (effects (font (size 1.27 1.27)))
     )
-    (property "Value" "10K 0805" (at 66.04 51.435 90) (show_name)
+    (property "Value" "Value: 10K 0805" (at 66.04 51.435 90) (show_name)
       (effects (font (size 1.27 1.27)))
     )
@@
       (effects (font (size 1.27 1.27)))
     )
-    (property "Value" "GW CSSRM3.CM-MFN4-A232-1-L" (at 113.03 69.215 0)
-      (effects (font (size 1.27 1.27)) hide)
-    )
+    (property "Value" "GW CSSRM1.BM" (at 113.03 69.215 0)
+      (effects (font (size 1.27 1.27)) hide)
+    )

Commit message: swapped around some parts and re-routed various bits and generated gerbers
Parts:
- removed D1, D2, D3: GW CSSRM1.BM, GW_CSSRM3:GW_CSSRM3, symbol GW CSSRM3:GW_CSSRM3
- added H1, H2: MountingHole, MountingHole:MountingHole_2.2mm_M2_DIN965_Pad, symbol Mechanical:MountingHole_Pad
- added LED1, LED2, LED3, LED4: KW H3L531.TE, KW_H3L531.TE:KW_H3L531.TE, symbol KW H3L531.TE:KW_H3L531.TE
- R2: value 170mΩ 2512 -> 190mΩ 2512
Connections:
- net GND: now also H1.1, H2.1
- net at C5.1, C6.1, L1.2: now also LED1.1 (Anode), LED1.2 (Anode), LED1.3 (Anode), LED2.1 (Anode), LED2.2 (Anode), LED2.3 (Anode), LED3.1 (Anode), LED3.2 (Anode), LED3.3 (Anode), LED4.1 (Anode), LED4.2 (Anode), LED4.3 (Anode)
- net at R2.1, U1.4 (VFB): now also LED1.4 (Cathode), LED1.5 (Cathode), LED1.6 (Cathode), LED2.4 (Cathode), LED2.5 (Cathode), LED2.6 (Cathode), LED3.4 (Cathode), LED3.5 (Cathode), LED3.6 (Cathode), LED4.4 (Cathode), LED4.5 (Cathode), LED4.6 (Cathode)

Commit message: swapped  the switch for pin headers so a switch can be wired externally to the PCB.
Parts:
- SW1: footprint Button_Switch_SMD:SW_SPDT_PCM12 -> Connector_Wire:SolderWire-0.1sqmm_1x03_P3.6mm_D0.4mm_OD1mm
Changed lines of the file:
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@@
       (effects (font (size 1.27 1.27)))
     )
-    (property "Footprint" "Button_Switch_SMD:SW_SPDT_PCM12" (at 40.005 43.815 0)
+    (property "Footprint" "Connector_Wire:SolderWire-0.1sqmm_1x03_P3.6mm_D0.4mm_OD1mm" (at 40.005 43.815 0)
       (effects (font (size 1.27 1.27)) hide)
     )

Commit message: Added new footprint for smaller cheaper, newer led.
Parts:
- removed LED1, LED2, LED3, LED4: KW H3L531.TE, KW_H3L531.TE:KW_H3L531.TE, symbol KW H3L531.TE:KW_H3L531.TE
- added LED1, LED2, LED3: KW_CDLMM2.TK-Y2Y6-4L16M1-2686, KW_CDLMM2.TK:KWCDLMM2TKY2Y64L16M12686, symbol KW_CDLMM2_TK-Y2Y6-4L16M1-2686:KW_CDLMM2.TK-Y2Y6-4L16M1-2686
- R2: value 190mΩ 2512 -> 1.1Ω 2512
Connections:
- net GND: now also LED1.3 (EP), LED2.3 (EP), LED3.3 (EP)
- net at C5.1, C6.1, L1.2: now also LED1.2 (A), LED2.2 (A), LED3.2 (A)
- net at R2.1, U1.4 (VFB): now also LED1.1 (K), LED2.1 (K), LED3.1 (K)
