File: KiCad files/LedBoard/LedBoard.kicad_pcb (KiCad board)
At the start: 2 copper layers, 40 x 40 mm, 18 parts, among them J4 7-5530843-7, Q1 IRLR120NTRPBF

Commit message: updated LED board to use new LEDs
Parts:
- removed C1, C5: 100nF, Capacitor_SMD:C_0805_2012Metric
- removed C2: 10uF 0805, Capacitor_SMD:C_0805_2012Metric
- removed C3: 100nF 0805, Capacitor_SMD:C_0805_2012Metric
- removed C4: 22uF, Capacitor_SMD:C_0805_2012Metric
- removed L1: MDA7030-2R2M, Inductor_SMD:L_Coilcraft_XAL7030-222
- removed LEDB1, LEDB3: GW VJLPL1.CM-K3LX-XX55-1, GWVJLPL1CMK3LXXX511:GWVJLPL1CMK3LXXX511
- removed PS1: TPS566242DRLR, Package_TO_SOT_SMD:SOT-563
- removed Q1: IRLR120NTRPBF, Package_TO_SOT_SMD:TO-252-2
- removed R1: 100K 0805, Resistor_SMD:R_0805_2012Metric
- removed R2: 120K 0805, Resistor_SMD:R_0805_2012Metric
- removed R3: 23.2K 0805, Resistor_SMD:R_0805_2012Metric
- removed R4: 30K 0805, Resistor_SMD:R_0805_2012Metric
- added LED10: L1505790500600000, L150-5790500600000:L1505790500600000, F.Cu at (104.5, 33.4)
- added LED11: L1505790500600000, L150-5790500600000:L1505790500600000, F.Cu at (75.5, 40.6)
- added LED12: L1505790500600000, L150-5790500600000:L1505790500600000, F.Cu at (82.8, 46.6)
- added LED13: L1505790500600000, L150-5790500600000:L1505790500600000, F.Cu at (90.0, 46.6)
- added LED14: L1505790500600000, L150-5790500600000:L1505790500600000, F.Cu at (97.2, 46.6)
- added LED15: L1505790500600000, L150-5790500600000:L1505790500600000, F.Cu at (104.5, 40.6)
- added LED16: L1505790500600000, L150-5790500600000:L1505790500600000, F.Cu at (75.5, 47.9)
- added LED17: L1505790500600000, L150-5790500600000:L1505790500600000, F.Cu at (82.8, 53.9)
- added LED18: L1505790500600000, L150-5790500600000:L1505790500600000, F.Cu at (90.0, 53.9)
- added LED19: L1505790500600000, L150-5790500600000:L1505790500600000, F.Cu at (97.2, 53.9)
- added LED20: L1505790500600000, L150-5790500600000:L1505790500600000, F.Cu at (104.5, 47.9)
- added LED4: L1505790500600000, L150-5790500600000:L1505790500600000, F.Cu at (97.2, 32.1)
- added LED5: L1505790500600000, L150-5790500600000:L1505790500600000, F.Cu at (104.5, 26.1)
- added LED6: L1505790500600000, L150-5790500600000:L1505790500600000, F.Cu at (75.5, 33.4)
- added LED7: L1505790500600000, L150-5790500600000:L1505790500600000, F.Cu at (82.8, 39.4)
- added LED8: L1505790500600000, L150-5790500600000:L1505790500600000, F.Cu at (90.0, 39.4)
- added LED9: L1505790500600000, L150-5790500600000:L1505790500600000, F.Cu at (97.2, 39.4)
- LED1, LED2, LED3: value GW VJLPL1.CM-K3LX-XX55-1 -> L1505790500600000; footprint GW_VJLPE1:GW_VJLPE1.CM_0.91x0.91mm -> L150-5790500600000:L1505790500600000
- moved LED2 17.2 mm to (82.8, 32.1), turned to 0 degrees
- moved LED1 9.74 mm to (75.5, 26.1), turned to 0 degrees
- moved LED3 4.88 mm to (90.0, 32.1), turned to 0 degrees
- moved J4 3.20 mm to (92.5, 22.9)
Connections:
- J4 pad 3: NPN GATE -> unconnected-(J4-Pad3)
- J4 pad 4: NPN GATE -> unconnected-(J4-Pad4)
- LED1 pad 1: NPN_DRAIN -> GND
- LED1 pad 2: LED_V+ -> VCC
- LED2 pad 1: NPN_DRAIN -> GND
- LED2 pad 2: LED_V+ -> VCC
- LED3 pad 1: NPN_DRAIN -> GND
- LED3 pad 2: LED_V+ -> VCC
Routing:
- net VCC: track 41.3 -> 198.8 mm
- net NPN GATE: track 25.2 -> 0.00 mm
- net LED_V+: track 15.7 -> 0.00 mm
- net GND: track 12.7 -> 0.00 mm
- net Net-(PS1-SW): track 12.0 -> 0.00 mm
- net Net-(PS1-FB): track 5.80 -> 0.00 mm
- net Net-(PS1-EN): track 5.08 -> 0.00 mm
- added copper zone on B.Cu, net GND
- removed copper zone on F.Cu, net LED_V+
- removed copper zone on F.Cu, net NPN_DRAIN
Other:
- board size 40 x 40 mm -> 46 x 46 mm
