File: KiCad files/EDC Size/EDC MainBoard/BQ25622ERYKR.kicad_sch (KiCad schematic)
At the start: 36 parts, among them IC1 BQ25638YBGR, J3 Conn_01x03, J4 Conn_01x02, J5 Conn_01x02, J6 Conn_01x02, J7 Conn_01x02, J8 Conn_01x02, J9 Conn_01x04, SW1 SW_Push, U2 BQ25622ERYKR

Commit message: updated the schematics and completed the battery charge IC circuit
Parts:
- added C25: 1uF 25V, Capacitor_SMD:C_0402_1005Metric, symbol Device:C_Small
- added C26, C29, C30, C31: 10uF 25V, Capacitor_SMD:C_0402_1005Metric, symbol Device:C_Small
- added C27, C32: 0.1uF 25V, Capacitor_SMD:C_0402_1005Metric, symbol Device:C_Small
- added C28: 47nF 25V, Capacitor_SMD:C_0402_1005Metric, symbol Device:C_Small
- added J11: Conn_01x02, Connector_PinHeader_2.54mm:PinHeader_1x02_P2.54mm_Vertical, symbol Connector_Generic:Conn_01x02
- added J12: Conn_01x03, Connector_PinHeader_2.54mm:PinHeader_1x03_P2.54mm_Vertical, symbol Connector_Generic:Conn_01x03
- added L3: SRP3212-1R0M, Inductor_SMD_Wurth:L_Wurth_WE-LQSH-3012, symbol Device:L_Small
- added R39: 820r 0402, Resistor_SMD:R_0402_1005Metric, symbol Device:R_Small
- added R40, R41: 10K 0402, Resistor_SMD:R_0402_1005Metric, symbol Device:R_Small
- added R43: 4.7K 0402, Resistor_SMD:R_0402_1005Metric, symbol Device:R_Small
- added SW2: SW_Push, Button_Switch_SMD:SW_SPST_B3U-1000P, symbol Switch:SW_Push
- added TP10, TP11, TP12, TP13, TP14: TestPoint, TestPoint:TestPoint_Pad_D1.0mm, symbol Connector:TestPoint
- C11, C12, C13, C14, C15, C16, C17, C18, IC1, J3, J4, L1, R21, R22, R23, R24, R25, SW1, TP5, TP6, TP7, TP8, TP9: now not fitted; now left out of the parts list
Connections:
- net CE: now also U2.14 (CE), R41.2
- net GND: now also U2.15 (GND), C25.2, C26.2, C27.2, C29.2, C30.2, C31.1, C32.2, J11.2 (Pin_2), J12.3 (Pin_3), R39.1, SW2.2, TP10.1, TP14.1
- net I2C_SCL: now also U2.13 (SCL), TP12.1
- net I2C_SDA: now also U2.12 (SDA), TP11.1
- net INT: now also U2.11 (*INT), R40.2, TP13.1
- net PG: now also U2.3 (*PG)
- net STAT: now also U2.10 (STAT)
- net SYS: now also U2.9 (SYS), C29.1, C30.1, J11.1 (Pin_1), L3.2, R40.1, R41.1
- net TS: now also U2.6 (TS), J12.2 (Pin_2)
- net TS_BIAS: now also U2.5 (TS_BIAS)
- net VSYS: now also U2.18 (VBUS), C25.1
- net at U2.1 (BTST): now also C28.2
- net at U2.16 (SW): now also C28.1, L3.1
- net at U2.17 (PMID): now also C26.1, C27.1
- net at U2.2 (REGN): now also C32.1
- net at U2.4 (ILIM): now also R39.2
- net at U2.7 (*QON): now also R43.1
- net at U2.8 (BAT): now also C31.2, J12.1 (Pin_1)
- new net: R43.2, SW2.1
