File: KiCad files/High Power Variant/ChargerPCB-PD-HP/ChargeBoard.kicad_sch (KiCad schematic)
At the start: 96 parts, among them IC1 BQ25792RQMR, IC2 TPS25750DRJKR, J1 HRO_TYPE-C-31-M-12, J10 3S/1.5MHz/1A ICGH, J11 4S/1.5MHz/1A ICGH, J3 Aardvark, J4 SYS/GND, J5 BAT/GND, J6 Aardvark, J7 THERMISTOR / GND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

Commit message: updated the schematics and completed the battery charge IC circuit
Changed lines of the file:
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@@
 	)
 	(junction
-		(at 266.7 167.005)
-		(diameter 0)
-		(color 0 0 0 0)
-	)
-	(junction
 		(at 353.06 127)
 		(diameter 0)
@@
 	(wire
 		(pts
-			(xy 392.43 121.92) (xy 389.255 121.92)
+			(xy 393.7 119.38) (xy 389.255 119.38)
 		)
 		(stroke
@@
 	(wire
 		(pts
-			(xy 392.43 124.46) (xy 389.255 124.46)
+			(xy 392.43 124.46) (xy 389.89 124.46)
 		)
 		(stroke
@@
 	(wire
 		(pts
-			(xy 389.255 124.46) (xy 389.255 121.92)
+			(xy 389.89 124.46) (xy 389.89 121.92)
 		)
 		(stroke
@@
 	(wire
 		(pts
-			(xy 266.065 167.005) (xy 266.7 167.005)
+			(xy 396.24 28.575) (xy 389.89 28.575)
 		)
 		(stroke
@@
 	(wire
 		(pts
-			(xy 396.24 28.575) (xy 389.89 28.575)
+			(xy 389.255 119.38) (xy 389.255 121.92)
 		)
 		(stroke
@@
 	(wire
 		(pts
+			(xy 389.89 121.92) (xy 389.255 121.92)
+		)
+		(stroke
+			(width 0)
+			(type default)
+		)
+	)
+	(wire
+		(pts
 			(xy 363.855 77.47) (xy 374.015 77.47)
 		)
@@
 	(text_box "ICs to look at for 240W EPR"
 		(exclude_from_sim no)
-		(at 20.32 180.975 0)
-		(size 30.48 10.795)
+		(at 12.7 302.895 0)
+		(size 33.02 19.685)
 		(stroke
 			(width 0)
@@
 	(text "Need to swap for BQ25731\neventually"
 		(exclude_from_sim no)
-		(at 287.02 92.71 0)
+		(at 16.51 317.5 0)
 		(effects
 			(font
 				(size 1.27 1.27)
-				(thickness 0.254)
-				(bold yes)
+				(thickness 0.1588)
 			)
 			(justify left bottom)
@@
 	(text "BQ25756E"
 		(exclude_from_sim no)
-		(at 26.67 189.23 0)
+		(at 21.59 311.15 0)
 		(effects
 			(font
@@
 	(text "TPS25751"
 		(exclude_from_sim no)
-		(at 26.67 186.69 0)
+		(at 21.59 308.61 0)
 		(effects
 			(font
@@
 	(global_label "SYS"
 		(shape input)
-		(at 392.43 121.92 0)
+		(at 393.7 119.38 0)
 		(fields_autoplaced yes)
 		(effects
@@
 		)
 		(property "Intersheetrefs" "${INTERSHEET_REFS}"
-			(at 398.9228 121.92 0)
+			(at 400.1928 119.38 0)
 			(effects
 				(font
@@
 		(dnp no)
 		(property "Reference" "D1"
-			(at 352.425 31.115 90)
+			(at 351.79 31.75 90)
 			(effects
 				(font
@@
 		)
 		(property "Value" "Diode, Schottky, 40 V, 5 A, SMC"
-			(at 351.79 32.385 90)
+			(at 349.885 34.925 90)
 			(effects
 				(font
 					(size 0.635 0.635)
 				)
-				(justify left)
 			)
 		)
@@
 		(dnp no)
 		(property "Reference" "C56"
-			(at 77.47 27.305 0)
+			(at 78.74 26.035 0)
 			(effects
 				(font
@@
 		)
 		(property "Value" "50V 0.01uF 0402 X7R"
-			(at 78.105 29.21 0)
+			(at 79.375 32.385 0)
 			(effects
 				(font
 					(size 0.5 0.5)
 				)
-				(justify left)
 			)
 		)
@@
 		(dnp no)
 		(property "Reference" "C55"
-			(at 71.755 27.305 0)
+			(at 73.025 26.035 0)
 			(effects
 				(font
@@
 		)
 		(property "Value" "50V 0.01uF 0402 X7R"
-			(at 72.39 29.21 0)
+			(at 73.66 31.115 0)
 			(effects
 				(font
 					(size 0.5 0.5)
 				)
-				(justify left)
 			)
 		)
@@
 		(dnp no)
 		(property "Reference" "C57"
-			(at 81.915 27.305 0)
+			(at 83.185 26.035 0)
 			(effects
 				(font
@@
 		)
 		(property "Value" "50V 0.01uF 0402 X7R"
-			(at 82.55 29.21 0)
+			(at 88.265 26.035 0)
 			(effects
 				(font
 					(size 0.5 0.5)
 				)
-				(justify left)
 			)
 		)
@@
 		(dnp no)
 		(property "Reference" "C53"
-			(at 60.325 27.305 0)
+			(at 61.595 26.035 0)
 			(effects
 				(font
@@
 		)
 		(property "Value" "50V 4.7uF 0603 X5R"
-			(at 60.96 29.21 0)
+			(at 62.23 31.75 0)
 			(effects
 				(font
 					(size 0.5 0.5)
 				)
-				(justify left)
 			)
 		)
@@
 		(dnp no)
 		(property "Reference" "C54"
-			(at 66.04 27.305 0)
+			(at 67.31 26.035 0)
 			(effects
 				(font
@@
 		)
 		(property "Value" "50V 0.01uF 0402 X7R"
-			(at 66.675 29.21 0)
+			(at 67.945 33.02 0)
 			(effects
 				(font
 					(size 0.5 0.5)
 				)
-				(justify left)
 			)
 		)
